File: EDA/mosfets.kicad_sch (KiCad schematic)
At the start: 44 parts, among them J10 Conn_01x04, J11 Conn_01x04, J12 Conn_01x04, J13 Conn_01x01, J14 Conn_01x01, J3 Conn_01x04, J4 Conn_01x04, J5 Conn_01x04, J6 Conn_01x04, J7 Conn_01x04, J8 Conn_01x04, J9 Conn_01x04, Q1 IRF4905STRLPBF, Q2 IRF4905STRLPBF, Q3 IRF4905STRLPBF, Q4 IRF4905STRLPBF, Q5 IRF4905STRLPBF, Q6 IRF4905STRLPBF, Q7 IRF4905STRLPBF, Q8 IRF4905STRLPBF, U10 PC817, U11 PC817, U4 PC817, U5 PC817, U6 PC817, U7 PC817, U8 PC817, U9 PC817

Commit message: Rename
Parts:
- added D1, D2, D3, D4, D5, D6, D7, D8: SS54, Diode_SMD:D_SMB, symbol Device:D_Schottky
- renumbered J6 to J1, J11 to J10, J3 to J11, J8 to J12, J5 to J2, J4 to J3, J10 to J4, J9 to J5, J7 to J6, J13 to J7, J14 to J8, J12 to J9, Q2 to Q1, Q3 to Q2, Q1 to Q3, Q6 to Q4, Q4 to Q6, Q8 to Q7, Q7 to Q8, R8 to R1, R17 to R10, R15 to R11, R13 to R12, R20 to R13, R18 to R14, R21 to R15, R19 to R16, R10 to R2, R7 to R3, R9 to R4, R11 to R5, R16 to R7, R14 to R8, R12 to R9, U5 to U1, U6 to U2, U4 to U3, U9 to U4, U8 to U5, U7 to U6, U11 to U7, U10 to U8
Connections:
- net +15V: now also D1.2 (A), D2.2 (A), D3.2 (A), D4.2 (A), D5.2 (A), D6.2 (A), D7.2 (A), D8.2 (A)
- net 12V_OUT01: now also D3.1 (K)
- net 12V_OUT02: now also D1.1 (K)
- net 12V_OUT03: now also D2.1 (K)
- net 12V_OUT04: now also D6.1 (K)
- net 12V_OUT05: now also D5.1 (K)
- net 12V_OUT06: now also D4.1 (K)
- net 12V_OUT07: now also D8.1 (K)
- net 12V_OUT08: now also D7.1 (K)
