File: EDA/trailcurrent-torrent.kicad_pcb (KiCad board)
At the start: 2 copper layers, 134.7 x 91.9 mm, 60 parts, among them IC1 AP63203WU-7, J1 Conn_01x06, J10 Conn_01x04, J11 Conn_01x04, J12 Conn_01x04, J13 Conn_01x01, J14 Conn_01x01, J2 Conn_01x04, J3 Conn_01x04, J4 Conn_01x04, J5 Conn_01x04, J6 Conn_01x04, J7 Conn_01x04, J8 Conn_01x04, J9 Conn_01x04, Q1 IRF4905STRLPBF, Q2 IRF4905STRLPBF, Q3 IRF4905STRLPBF, Q4 IRF4905STRLPBF, Q5 IRF4905STRLPBF, Q6 IRF4905STRLPBF, Q7 IRF4905STRLPBF, Q8 IRF4905STRLPBF, SW1 SW_DIP_x04, U1 ESP32-WROOM-32, U10 PC817, U11 PC817, U2 SN65HVD230, U4 PC817, U5 PC817, U6 PC817, U7 PC817, U8 PC817, U9 PC817

Commit message: Rename
Parts:
- added D1: SS54, Diode_SMD:D_SMB, F.Cu at (38.3, 79.4)
- added D2: SS54, Diode_SMD:D_SMB, F.Cu at (59.0, 145.3)
- added D3: SS54, Diode_SMD:D_SMB, F.Cu at (59.0, 150.8)
- added D4: SS54, Diode_SMD:D_SMB, F.Cu at (59.0, 156.4)
- added D5: SS54, Diode_SMD:D_SMB, F.Cu at (59.0, 161.9)
- added D6: SS54, Diode_SMD:D_SMB, F.Cu at (59.0, 167.5)
- added D7: SS54, Diode_SMD:D_SMB, F.Cu at (59.0, 173.0)
- added D8: SS54, Diode_SMD:D_SMB, F.Cu at (59.0, 178.6)
Routing:
- net +15V: track 16.8 -> 24.8 mm
